Commit message: added gazebo support for the IRB 120T varient. Reverted link masses back to those given in solidworks

File: abb_irb120_support/urdf/irb120t_gazebo_macro.xacro (robot description, xacro)
@@ -1,5 +1,5 @@
 <?xml version="1.0"?>
 <robot xmlns:xacro="http://ros.org/wiki/xacro">
-<xacro:macro name="abb_irb120" params="prefix">
+<xacro:macro name="abb_irb120t" params="prefix">
   <!-- link list -->
   <link name="${prefix}base_link">
@@ -187,5 +187,5 @@
     <parent link="${prefix}link_3"/>
     <child link="${prefix}link_4"/>
-    <limit effort="30" lower="-2.79253" upper="2.79253" velocity="5.58505"/>
+    <limit effort="30" lower="-2.79253" upper="2.79253" velocity="7.33038"/>
     <axis xyz="1 0 0"/>
     <dynamics damping="0.0" friction="0.0"/>
@@ -195,5 +195,5 @@
     <parent link="${prefix}link_4"/>
     <child link="${prefix}link_5"/>
-    <limit effort="30" lower="-2.094395" upper="2.094395" velocity="5.58505"/>
+    <limit effort="30" lower="-2.094395" upper="2.094395" velocity="10.29744"/>
     <axis xyz="0 1 0"/>
     <dynamics damping="0.0" friction="0.0"/>
@@ -203,5 +203,5 @@
     <parent link="${prefix}link_5"/>
     <child link="${prefix}link_6"/>
-    <limit effort="30" lower="-6.98132" upper="6.98132" velocity="7.33038"/>
+    <limit effort="30" lower="-6.98132" upper="6.98132" velocity="10.471975"/>
     <axis xyz="1 0 0"/>
     <dynamics damping="0.0" friction="0.0"/>
