Commit message: reduced decimal places of inertial properties, added instructions for controlling gazebo model using moveit

File: abb_irb120_support/urdf/irb120_gazebo_macro.xacro (robot description, xacro)
@@ -6,6 +6,6 @@
     <inertial>
       <mass value="6.215"/>
-      <origin xyz="-0.042039286 8.0131669E-05 0.079637532" rpy="0 0 0"/>
-      <inertia ixx="0.024727161" ixy="-8.078424E-05" ixz="0.0013090238" iyy="0.049128491" iyz="-8.0419046E-06" izz="0.047237615"/>
+      <origin xyz="-0.04204 8.01E-05 0.07964" rpy="0 0 0"/>
+      <inertia ixx="0.0247272" ixy="-8.0784E-05" ixz="0.00130902" iyy="0.0491285" iyz="-8.0419E-06" izz="0.0472376"/>
     </inertial>
     <visual>
@@ -31,6 +31,6 @@
     <inertial>
       <mass value="3.067" />
-      <origin xyz="9.7686412E-05 -0.00011929533 0.23841183" rpy="0 0 0"/>
-      <inertia ixx="0.014217456" ixy="-1.2857888E-05" ixz="-2.3136423E-05" iyy="0.014404147" iyz="1.9340368E-05" izz="0.010453301"/>
+      <origin xyz="9.77E-05 -0.00012 0.23841" rpy="0 0 0"/>
+      <inertia ixx="0.0142175" ixy="-1.28579E-05" ixz="-2.31364E-05" iyy="0.0144041" iyz="1.93404E-05" izz="0.0104533"/>
     </inertial>
     <visual>
@@ -51,7 +51,7 @@
   <link name="${prefix}link_2">
     <inertial>
-      <mass value="3.908667"/>
-      <origin xyz="0.00077829178 -0.0021170276 0.1012432" rpy="0 0 0"/>
-      <inertia ixx="0.060311109" ixy="9.8343135E-06" ixz="5.7240689E-05" iyy="0.04156899" iyz="-0.00050497005" izz="0.025954849"/>
+      <mass value="3.9087"/>
+      <origin xyz="0.00078 -0.00212 0.10124" rpy="0 0 0"/>
+      <inertia ixx="0.0603111" ixy="9.83431E-06" ixz="5.72407E-05" iyy="0.041569" iyz="-0.00050497" izz="0.0259548"/>
     </inertial>
     <visual>
@@ -73,6 +73,6 @@
     <inertial>
       <mass value="2.94372"/>
-      <origin xyz="0.022807656 0.0010643596 0.057910651" rpy="0 0 0"/>
-      <inertia ixx="0.0083560552" ixy="-8.0154465E-05" ixz="0.0014288355" iyy="0.016712978" iyz="-0.00018222659" izz="0.012698447"/>
+      <origin xyz="0.02281 0.00106 0.05791" rpy="0 0 0"/>
+      <inertia ixx="0.00835606" ixy="-8.01545E-05" ixz="0.00142884" iyy="0.016713" iyz="-0.000182227" izz="0.0126984"/>
     </inertial>
     <visual>
@@ -94,6 +94,6 @@
     <inertial>
       <mass value="1.3278642"/>
-      <origin xyz="0.22470384 0.00015341817 0.00040552537" rpy="0 0 0"/>
-      <inertia ixx="0.0028466109" ixy="-2.1276535E-05" ixz="-1.643522E-05" iyy="0.0040134585" iyz="1.313359E-05" izz="0.0052535097"/>
+      <origin xyz="0.2247 0.00015 0.00041" rpy="0 0 0"/>
+      <inertia ixx="0.00284661" ixy="-2.12765E-05" ixz="-1.6435E-05" iyy="0.00401346" iyz="1.31336E-05" izz="0.0052535"/>
     </inertial>
     <visual>
@@ -115,6 +115,6 @@
     <inertial>
       <mass value="0.54662685"/>
-      <origin xyz="-0.0010948374 3.6852479E-05 6.2216732E-05" rpy="0 0 0"/>
-      <inertia ixx="0.00040489103" ixy="1.6194294E-06" ixz="8.4680493E-07" iyy="0.00089282497" iyz="-1.5179204E-08" izz="0.00081546839"/>
+      <origin xyz="-0.00109 3.68E-05 6.22E-05" rpy="0 0 0"/>
+      <inertia ixx="0.000404891" ixy="1.61943E-06" ixz="8.46805E-07" iyy="0.000892825" iyz="-1.51792E-08" izz="0.000815468"/>
     </inertial>
     <visual>
@@ -136,5 +136,5 @@
     <inertial>
       <mass value="0.01367842"/>
-      <origin xyz="-0.0070620873 -0.00016958101 -1.3236698E-06" rpy="0 0 0"/>
+      <origin xyz="-0.00706 -0.00017 -1.32E-06" rpy="0 0 0"/>
       <inertia ixx="0.001" ixy="0" ixz="0" iyy="0.001" iyz="0" izz="0.001"/>
     </inertial>

Commit message: updated moveit package to accept gazebo argument. Increased link masses proportionally to reach 25kg (as specified on ABB website)

File: abb_irb120_support/urdf/irb120_gazebo_macro.xacro (robot description, xacro)
@@ -5,5 +5,5 @@
   <link name="${prefix}base_link">
     <inertial>
-      <mass value="6.215"/>
+      <mass value="8.562"/>
       <origin xyz="-0.04204 8.01E-05 0.07964" rpy="0 0 0"/>
       <inertia ixx="0.0247272" ixy="-8.0784E-05" ixz="0.00130902" iyy="0.0491285" iyz="-8.0419E-06" izz="0.0472376"/>
@@ -30,5 +30,5 @@
   <link name="${prefix}link_1">
     <inertial>
-      <mass value="3.067" />
+      <mass value="4.225" />
       <origin xyz="9.77E-05 -0.00012 0.23841" rpy="0 0 0"/>
       <inertia ixx="0.0142175" ixy="-1.28579E-05" ixz="-2.31364E-05" iyy="0.0144041" iyz="1.93404E-05" izz="0.0104533"/>
@@ -51,5 +51,5 @@
   <link name="${prefix}link_2">
     <inertial>
-      <mass value="3.9087"/>
+      <mass value="5.385"/>
       <origin xyz="0.00078 -0.00212 0.10124" rpy="0 0 0"/>
       <inertia ixx="0.0603111" ixy="9.83431E-06" ixz="5.72407E-05" iyy="0.041569" iyz="-0.00050497" izz="0.0259548"/>
@@ -72,5 +72,5 @@
   <link name="${prefix}link_3">
     <inertial>
-      <mass value="2.94372"/>
+      <mass value="4.056"/>
       <origin xyz="0.02281 0.00106 0.05791" rpy="0 0 0"/>
       <inertia ixx="0.00835606" ixy="-8.01545E-05" ixz="0.00142884" iyy="0.016713" iyz="-0.000182227" izz="0.0126984"/>
@@ -93,5 +93,5 @@
   <link name="${prefix}link_4">
     <inertial>
-      <mass value="1.3278642"/>
+      <mass value="1.83"/>
       <origin xyz="0.2247 0.00015 0.00041" rpy="0 0 0"/>
       <inertia ixx="0.00284661" ixy="-2.12765E-05" ixz="-1.6435E-05" iyy="0.00401346" iyz="1.31336E-05" izz="0.0052535"/>
@@ -114,5 +114,5 @@
   <link name="${prefix}link_5">
     <inertial>
-      <mass value="0.54662685"/>
+      <mass value="0.752"/>
       <origin xyz="-0.00109 3.68E-05 6.22E-05" rpy="0 0 0"/>
       <inertia ixx="0.000404891" ixy="1.61943E-06" ixz="8.46805E-07" iyy="0.000892825" iyz="-1.51792E-08" izz="0.000815468"/>
@@ -135,5 +135,5 @@
   <link name="${prefix}link_6">
     <inertial>
-      <mass value="0.01367842"/>
+      <mass value="0.189"/>
       <origin xyz="-0.00706 -0.00017 -1.32E-06" rpy="0 0 0"/>
       <inertia ixx="0.001" ixy="0" ixz="0" iyy="0.001" iyz="0" izz="0.001"/>

Commit message: updated to use position controllers in gazebo simulation

File: abb_irb120_support/urdf/irb120_gazebo_macro.xacro (robot description, xacro)
@@ -163,5 +163,5 @@
     <parent link="${prefix}base_link"/>
     <child link="${prefix}link_1"/>
-    <limit effort="100" lower="-2.87979" upper="2.87979" velocity="4.36332"/>
+    <limit effort="0" lower="-2.87979" upper="2.87979" velocity="4.36332"/>
     <axis xyz="0 0 1"/>
     <dynamics damping="0.0" friction="0.0"/>
@@ -171,5 +171,5 @@
     <parent link="${prefix}link_1"/>
     <child link="${prefix}link_2"/>
-    <limit effort="100" lower="-1.91986" upper="1.91986" velocity="4.36332"/>
+    <limit effort="0" lower="-1.91986" upper="1.91986" velocity="4.36332"/>
     <axis xyz="0 1 0"/>
     <dynamics damping="0.0" friction="0.0"/>
@@ -179,5 +179,5 @@
     <parent link="${prefix}link_2"/>
     <child link="${prefix}link_3"/>
-    <limit effort="100" lower="-1.91986" upper="1.22173" velocity="4.36332"/>
+    <limit effort="0" lower="-1.91986" upper="1.22173" velocity="4.36332"/>
     <axis xyz="0 1 0"/>
     <dynamics damping="0.0" friction="0.0"/>
@@ -187,5 +187,5 @@
     <parent link="${prefix}link_3"/>
     <child link="${prefix}link_4"/>
-    <limit effort="30" lower="-2.79253" upper="2.79253" velocity="5.58505"/>
+    <limit effort="0" lower="-2.79253" upper="2.79253" velocity="5.58505"/>
     <axis xyz="1 0 0"/>
     <dynamics damping="0.0" friction="0.0"/>
@@ -195,5 +195,5 @@
     <parent link="${prefix}link_4"/>
     <child link="${prefix}link_5"/>
-    <limit effort="30" lower="-2.094395" upper="2.094395" velocity="5.58505"/>
+    <limit effort="0" lower="-2.094395" upper="2.094395" velocity="5.58505"/>
     <axis xyz="0 1 0"/>
     <dynamics damping="0.0" friction="0.0"/>
@@ -203,5 +203,5 @@
     <parent link="${prefix}link_5"/>
     <child link="${prefix}link_6"/>
-    <limit effort="30" lower="-6.98132" upper="6.98132" velocity="7.33038"/>
+    <limit effort="0" lower="-6.98132" upper="6.98132" velocity="7.33038"/>
     <axis xyz="1 0 0"/>
     <dynamics damping="0.0" friction="0.0"/>
@@ -223,9 +223,7 @@
   <transmission name="${prefix}tran1">
     <type>transmission_interface/SimpleTransmission</type>
-    <joint name="${prefix}joint_1">
-      <hardwareInterface>EffortJointInterface</hardwareInterface>
-    </joint>
+    <joint name="${prefix}joint_1"/>
     <actuator name="${prefix}motor1">
-      <hardwareInterface>EffortJointInterface</hardwareInterface>
+      <hardwareInterface>PositionJointInterface</hardwareInterface>
       <mechanicalReduction>1</mechanicalReduction>
     </actuator>
@@ -233,9 +231,7 @@
   <transmission name="${prefix}tran2">
     <type>transmission_interface/SimpleTransmission</type>
-    <joint name="${prefix}joint_2">
-      <hardwareInterface>EffortJointInterface</hardwareInterface>
-    </joint>
+    <joint name="${prefix}joint_2"/>
     <actuator name="${prefix}motor2">
-      <hardwareInterface>EffortJointInterface</hardwareInterface>
+      <hardwareInterface>PositionJointInterface</hardwareInterface>
       <mechanicalReduction>1</mechanicalReduction>
     </actuator>
@@ -243,9 +239,7 @@
   <transmission name="${prefix}tran3">
     <type>transmission_interface/SimpleTransmission</type>
-    <joint name="${prefix}joint_3">
-      <hardwareInterface>EffortJointInterface</hardwareInterface>
-    </joint>
+    <joint name="${prefix}joint_3"/>
     <actuator name="${prefix}motor3">
-      <hardwareInterface>EffortJointInterface</hardwareInterface>
+      <hardwareInterface>PositionJointInterface</hardwareInterface>
       <mechanicalReduction>1</mechanicalReduction>
     </actuator>
@@ -253,9 +247,7 @@
   <transmission name="${prefix}tran4">
     <type>transmission_interface/SimpleTransmission</type>
-    <joint name="${prefix}joint_4">
-      <hardwareInterface>EffortJointInterface</hardwareInterface>
-    </joint>
+    <joint name="${prefix}joint_4"/>
     <actuator name="${prefix}motor4">
-      <hardwareInterface>EffortJointInterface</hardwareInterface>
+      <hardwareInterface>PositionJointInterface</hardwareInterface>
       <mechanicalReduction>1</mechanicalReduction>
     </actuator>
@@ -263,9 +255,7 @@
   <transmission name="${prefix}tran5">
     <type>transmission_interface/SimpleTransmission</type>
-    <joint name="${prefix}joint_5">
-      <hardwareInterface>EffortJointInterface</hardwareInterface>
-    </joint>
+    <joint name="${prefix}joint_5"/>
     <actuator name="${prefix}motor5">
-      <hardwareInterface>EffortJointInterface</hardwareInterface>
+      <hardwareInterface>PositionJointInterface</hardwareInterface>
       <mechanicalReduction>1</mechanicalReduction>
     </actuator>
@@ -273,9 +263,7 @@
   <transmission name="${prefix}tran6">
     <type>transmission_interface/SimpleTransmission</type>
-    <joint name="${prefix}joint_6">
-      <hardwareInterface>EffortJointInterface</hardwareInterface>
-    </joint>
+    <joint name="${prefix}joint_6"/>
     <actuator name="${prefix}motor6">
-      <hardwareInterface>EffortJointInterface</hardwareInterface>
+      <hardwareInterface>PositionJointInterface</hardwareInterface>
       <mechanicalReduction>1</mechanicalReduction>
     </actuator>

File: abb_irb120_support/urdf/irb120t_gazebo_macro.xacro (robot description, xacro)
@@ -163,5 +163,5 @@
     <parent link="${prefix}base_link"/>
     <child link="${prefix}link_1"/>
-    <limit effort="100" lower="-2.87979" upper="2.87979" velocity="4.36332"/>
+    <limit effort="0" lower="-2.87979" upper="2.87979" velocity="4.36332"/>
     <axis xyz="0 0 1"/>
     <dynamics damping="0.0" friction="0.0"/>
@@ -171,5 +171,5 @@
     <parent link="${prefix}link_1"/>
     <child link="${prefix}link_2"/>
-    <limit effort="100" lower="-1.91986" upper="1.91986" velocity="4.36332"/>
+    <limit effort="0" lower="-1.91986" upper="1.91986" velocity="4.36332"/>
     <axis xyz="0 1 0"/>
     <dynamics damping="0.0" friction="0.0"/>
@@ -179,5 +179,5 @@
     <parent link="${prefix}link_2"/>
     <child link="${prefix}link_3"/>
-    <limit effort="100" lower="-1.91986" upper="1.22173" velocity="4.36332"/>
+    <limit effort="0" lower="-1.91986" upper="1.22173" velocity="4.36332"/>
     <axis xyz="0 1 0"/>
     <dynamics damping="0.0" friction="0.0"/>
@@ -187,5 +187,5 @@
     <parent link="${prefix}link_3"/>
     <child link="${prefix}link_4"/>
-    <limit effort="30" lower="-2.79253" upper="2.79253" velocity="7.33038"/>
+    <limit effort="0" lower="-2.79253" upper="2.79253" velocity="7.33038"/>
     <axis xyz="1 0 0"/>
     <dynamics damping="0.0" friction="0.0"/>
@@ -195,5 +195,5 @@
     <parent link="${prefix}link_4"/>
     <child link="${prefix}link_5"/>
-    <limit effort="30" lower="-2.094395" upper="2.094395" velocity="10.29744"/>
+    <limit effort="0" lower="-2.094395" upper="2.094395" velocity="10.29744"/>
     <axis xyz="0 1 0"/>
     <dynamics damping="0.0" friction="0.0"/>
@@ -203,5 +203,5 @@
     <parent link="${prefix}link_5"/>
     <child link="${prefix}link_6"/>
-    <limit effort="30" lower="-6.98132" upper="6.98132" velocity="10.471975"/>
+    <limit effort="0" lower="-6.98132" upper="6.98132" velocity="10.471975"/>
     <axis xyz="1 0 0"/>
     <dynamics damping="0.0" friction="0.0"/>
@@ -223,9 +223,7 @@
   <transmission name="${prefix}tran1">
     <type>transmission_interface/SimpleTransmission</type>
-    <joint name="${prefix}joint_1">
-      <hardwareInterface>EffortJointInterface</hardwareInterface>
-    </joint>
+    <joint name="${prefix}joint_1"/>
     <actuator name="${prefix}motor1">
-      <hardwareInterface>EffortJointInterface</hardwareInterface>
+      <hardwareInterface>PositionJointInterface</hardwareInterface>
       <mechanicalReduction>1</mechanicalReduction>
     </actuator>
@@ -233,9 +231,7 @@
   <transmission name="${prefix}tran2">
     <type>transmission_interface/SimpleTransmission</type>
-    <joint name="${prefix}joint_2">
-      <hardwareInterface>EffortJointInterface</hardwareInterface>
-    </joint>
+    <joint name="${prefix}joint_2"/>
     <actuator name="${prefix}motor2">
-      <hardwareInterface>EffortJointInterface</hardwareInterface>
+      <hardwareInterface>PositionJointInterface</hardwareInterface>
       <mechanicalReduction>1</mechanicalReduction>
     </actuator>
@@ -243,9 +239,7 @@
   <transmission name="${prefix}tran3">
     <type>transmission_interface/SimpleTransmission</type>
-    <joint name="${prefix}joint_3">
-      <hardwareInterface>EffortJointInterface</hardwareInterface>
-    </joint>
+    <joint name="${prefix}joint_3"/>
     <actuator name="${prefix}motor3">
-      <hardwareInterface>EffortJointInterface</hardwareInterface>
+      <hardwareInterface>PositionJointInterface</hardwareInterface>
       <mechanicalReduction>1</mechanicalReduction>
     </actuator>
@@ -253,9 +247,7 @@
   <transmission name="${prefix}tran4">
     <type>transmission_interface/SimpleTransmission</type>
-    <joint name="${prefix}joint_4">
-      <hardwareInterface>EffortJointInterface</hardwareInterface>
-    </joint>
+    <joint name="${prefix}joint_4"/>
     <actuator name="${prefix}motor4">
-      <hardwareInterface>EffortJointInterface</hardwareInterface>
+      <hardwareInterface>PositionJointInterface</hardwareInterface>
       <mechanicalReduction>1</mechanicalReduction>
     </actuator>
@@ -263,9 +255,7 @@
   <transmission name="${prefix}tran5">
     <type>transmission_interface/SimpleTransmission</type>
-    <joint name="${prefix}joint_5">
-      <hardwareInterface>EffortJointInterface</hardwareInterface>
-    </joint>
+    <joint name="${prefix}joint_5"/>
     <actuator name="${prefix}motor5">
-      <hardwareInterface>EffortJointInterface</hardwareInterface>
+      <hardwareInterface>PositionJointInterface</hardwareInterface>
       <mechanicalReduction>1</mechanicalReduction>
     </actuator>
@@ -273,9 +263,7 @@
   <transmission name="${prefix}tran6">
     <type>transmission_interface/SimpleTransmission</type>
-    <joint name="${prefix}joint_6">
-      <hardwareInterface>EffortJointInterface</hardwareInterface>
-    </joint>
+    <joint name="${prefix}joint_6"/>
     <actuator name="${prefix}motor6">
-      <hardwareInterface>EffortJointInterface</hardwareInterface>
+      <hardwareInterface>PositionJointInterface</hardwareInterface>
       <mechanicalReduction>1</mechanicalReduction>
     </actuator>
