Commit message: Move Gazebo xacros to IRB 120 Gazebo pkg.
Also:
 - re-add inertial and dynamics tags to base xacro macros (these properties
   have to be included directly, as they cannot be added later using a
   "gazebo reference=''" tag)
 - update corresponding urdfs

File: abb_irb120_gazebo/urdf/irb120.xacro (robot description, xacro)
@@ -1,5 +1,5 @@
 <?xml version="1.0" ?>
 <robot name="abb_irb120" xmlns:xacro="http://ros.org/wiki/xacro">
-  <xacro:include filename="$(find abb_irb120_support)/urdf/irb120_gazebo_macro.xacro"/>
+  <xacro:include filename="$(find abb_irb120_gazebo)/urdf/irb120_macro.xacro"/>
   <xacro:abb_irb120 prefix=""/>
 </robot>

File: abb_irb120_gazebo/urdf/irb120t.xacro (robot description, xacro)
@@ -1,5 +1,5 @@
 <?xml version="1.0" ?>
 <robot name="abb_irb120t" xmlns:xacro="http://ros.org/wiki/xacro">
-  <xacro:include filename="$(find abb_irb120_support)/urdf/irb120t_gazebo_macro.xacro"/>
+  <xacro:include filename="$(find abb_irb120_gazebo)/urdf/irb120t_macro.xacro"/>
   <xacro:abb_irb120t prefix=""/>
 </robot>

File: abb_irb120_support/urdf/irb120.urdf (robot description, URDF)
Before this commit: robot abb_irb120, 9 links, 8 joints
Links:
- link base_link: mass None -> 6.215
- link link_1: mass None -> 3.067
- link link_2: mass None -> 3.909
- link link_3: mass None -> 2.944
- link link_4: mass None -> 1.328
- link link_5: mass None -> 0.546
- link link_6: mass None -> 0.137

File: abb_irb120_support/urdf/irb120_macro.xacro (robot description, xacro)
@@ -4,4 +4,9 @@
   <!-- link list -->
   <link name="${prefix}base_link">
+    <inertial>
+      <mass value="6.215"/>
+      <origin xyz="-0.04204 8.01E-05 0.07964" rpy="0 0 0"/>
+      <inertia ixx="0.0247272" ixy="-8.0784E-05" ixz="0.00130902" iyy="0.0491285" iyz="-8.0419E-06" izz="0.0472376"/>
+    </inertial>
     <visual>
       <origin xyz="0 0 0" rpy="0 0 0"/>
@@ -24,4 +29,9 @@
   </link>
   <link name="${prefix}link_1">
+    <inertial>
+      <mass value="3.067" />
+      <origin xyz="9.77E-05 -0.00012 0.23841" rpy="0 0 0"/>
+      <inertia ixx="0.0142175" ixy="-1.28579E-05" ixz="-2.31364E-05" iyy="0.0144041" iyz="1.93404E-05" izz="0.0104533"/>
+    </inertial>
     <visual>
       <origin xyz="0 0 0" rpy="0 0 0"/>
@@ -40,4 +50,9 @@
   </link>
   <link name="${prefix}link_2">
+    <inertial>
+      <mass value="3.909"/>
+      <origin xyz="0.00078 -0.00212 0.10124" rpy="0 0 0"/>
+      <inertia ixx="0.0603111" ixy="9.83431E-06" ixz="5.72407E-05" iyy="0.041569" iyz="-0.00050497" izz="0.0259548"/>
+    </inertial>
     <visual>
       <origin xyz="0 0 0" rpy="0 0 0"/>
@@ -56,4 +71,9 @@
   </link>
   <link name="${prefix}link_3">
+    <inertial>
+      <mass value="2.944"/>
+      <origin xyz="0.02281 0.00106 0.05791" rpy="0 0 0"/>
+      <inertia ixx="0.00835606" ixy="-8.01545E-05" ixz="0.00142884" iyy="0.016713" iyz="-0.000182227" izz="0.0126984"/>
+    </inertial>
     <visual>
       <origin xyz="0 0 0" rpy="0 0 0"/>
@@ -72,4 +92,9 @@
   </link>
   <link name="${prefix}link_4">
+    <inertial>
+      <mass value="1.328"/>
+      <origin xyz="0.2247 0.00015 0.00041" rpy="0 0 0"/>
+      <inertia ixx="0.00284661" ixy="-2.12765E-05" ixz="-1.6435E-05" iyy="0.00401346" iyz="1.31336E-05" izz="0.0052535"/>
+    </inertial>
     <visual>
       <origin xyz="0 0 0" rpy="0 0 0"/>
@@ -88,4 +113,9 @@
   </link>
   <link name="${prefix}link_5">
+    <inertial>
+      <mass value="0.546"/>
+      <origin xyz="-0.00109 3.68E-05 6.22E-05" rpy="0 0 0"/>
+      <inertia ixx="0.000404891" ixy="1.61943E-06" ixz="8.46805E-07" iyy="0.000892825" iyz="-1.51792E-08" izz="0.000815468"/>
+    </inertial>
     <visual>
       <origin xyz="0 0 0" rpy="0 0 0"/>
@@ -104,4 +134,9 @@
   </link>
   <link name="${prefix}link_6">
+    <inertial>
+      <mass value="0.137"/>
+      <origin xyz="-0.00706 -0.00017 -1.32E-06" rpy="0 0 0"/>
+      <inertia ixx="0.001" ixy="0" ixz="0" iyy="0.001" iyz="0" izz="0.001"/>
+    </inertial>
     <visual>
       <origin xyz="0 0 0" rpy="0 0 0"/>
@@ -130,4 +165,5 @@
     <limit effort="0" lower="-2.87979" upper="2.87979" velocity="4.36332"/>
     <axis xyz="0 0 1"/>
+    <dynamics damping="0.0" friction="0.0"/>
   </joint>
   <joint name="${prefix}joint_2" type="revolute">
@@ -137,4 +173,5 @@
     <limit effort="0" lower="-1.91986" upper="1.91986" velocity="4.36332"/>
     <axis xyz="0 1 0"/>
+    <dynamics damping="0.0" friction="0.0"/>
   </joint>
   <joint name="${prefix}joint_3" type="revolute">
@@ -144,4 +181,5 @@
     <limit effort="0" lower="-1.91986" upper="1.22173" velocity="4.36332"/>
     <axis xyz="0 1 0"/>
+    <dynamics damping="0.0" friction="0.0"/>
   </joint>
   <joint name="${prefix}joint_4" type="revolute">
@@ -151,4 +189,5 @@
     <limit effort="0" lower="-2.79253" upper="2.79253" velocity="5.58505"/>
     <axis xyz="1 0 0"/>
+    <dynamics damping="0.0" friction="0.0"/>
   </joint>
   <joint name="${prefix}joint_5" type="revolute">
@@ -158,4 +197,5 @@
     <limit effort="0" lower="-2.094395" upper="2.094395" velocity="5.58505"/>
     <axis xyz="0 1 0"/>
+    <dynamics damping="0.0" friction="0.0"/>
   </joint>
   <joint name="${prefix}joint_6" type="revolute">
@@ -165,4 +205,5 @@
     <limit effort="0" lower="-6.98132" upper="6.98132" velocity="7.33038"/>
     <axis xyz="1 0 0"/>
+    <dynamics damping="0.0" friction="0.0"/>
   </joint>
   <joint name="${prefix}joint6-tool0" type="fixed">

File: abb_irb120_support/urdf/irb120t.urdf (robot description, URDF)
Before this commit: robot abb_irb120t, 9 links, 8 joints
Links:
- link base_link: mass None -> 6.215
- link link_1: mass None -> 3.067
- link link_2: mass None -> 3.909
- link link_3: mass None -> 2.944
- link link_4: mass None -> 1.328
- link link_5: mass None -> 0.546
- link link_6: mass None -> 0.137

File: abb_irb120_support/urdf/irb120t_macro.xacro (robot description, xacro)
@@ -4,4 +4,9 @@
   <!-- link list -->
   <link name="${prefix}base_link">
+    <inertial>
+      <mass value="6.215"/>
+      <origin xyz="-0.04204 8.01E-05 0.07964" rpy="0 0 0"/>
+      <inertia ixx="0.0247272" ixy="-8.0784E-05" ixz="0.00130902" iyy="0.0491285" iyz="-8.0419E-06" izz="0.0472376"/>
+    </inertial>
     <visual>
       <origin xyz="0 0 0" rpy="0 0 0"/>
@@ -24,4 +29,9 @@
   </link>
   <link name="${prefix}link_1">
+    <inertial>
+      <mass value="3.067" />
+      <origin xyz="9.77E-05 -0.00012 0.23841" rpy="0 0 0"/>
+      <inertia ixx="0.0142175" ixy="-1.28579E-05" ixz="-2.31364E-05" iyy="0.0144041" iyz="1.93404E-05" izz="0.0104533"/>
+    </inertial>
     <visual>
       <origin xyz="0 0 0" rpy="0 0 0"/>
@@ -40,4 +50,9 @@
   </link>
   <link name="${prefix}link_2">
+    <inertial>
+      <mass value="3.909"/>
+      <origin xyz="0.00078 -0.00212 0.10124" rpy="0 0 0"/>
+      <inertia ixx="0.0603111" ixy="9.83431E-06" ixz="5.72407E-05" iyy="0.041569" iyz="-0.00050497" izz="0.0259548"/>
+    </inertial>
     <visual>
       <origin xyz="0 0 0" rpy="0 0 0"/>
@@ -56,4 +71,9 @@
   </link>
   <link name="${prefix}link_3">
+    <inertial>
+      <mass value="2.944"/>
+      <origin xyz="0.02281 0.00106 0.05791" rpy="0 0 0"/>
+      <inertia ixx="0.00835606" ixy="-8.01545E-05" ixz="0.00142884" iyy="0.016713" iyz="-0.000182227" izz="0.0126984"/>
+    </inertial>
     <visual>
       <origin xyz="0 0 0" rpy="0 0 0"/>
@@ -72,4 +92,9 @@
   </link>
   <link name="${prefix}link_4">
+    <inertial>
+      <mass value="1.328"/>
+      <origin xyz="0.2247 0.00015 0.00041" rpy="0 0 0"/>
+      <inertia ixx="0.00284661" ixy="-2.12765E-05" ixz="-1.6435E-05" iyy="0.00401346" iyz="1.31336E-05" izz="0.0052535"/>
+    </inertial>
     <visual>
       <origin xyz="0 0 0" rpy="0 0 0"/>
@@ -88,4 +113,9 @@
   </link>
   <link name="${prefix}link_5">
+    <inertial>
+      <mass value="0.546"/>
+      <origin xyz="-0.00109 3.68E-05 6.22E-05" rpy="0 0 0"/>
+      <inertia ixx="0.000404891" ixy="1.61943E-06" ixz="8.46805E-07" iyy="0.000892825" iyz="-1.51792E-08" izz="0.000815468"/>
+    </inertial>
     <visual>
       <origin xyz="0 0 0" rpy="0 0 0"/>
@@ -104,4 +134,9 @@
   </link>
   <link name="${prefix}link_6">
+    <inertial>
+      <mass value="0.137"/>
+      <origin xyz="-0.00706 -0.00017 -1.32E-06" rpy="0 0 0"/>
+      <inertia ixx="0.001" ixy="0" ixz="0" iyy="0.001" iyz="0" izz="0.001"/>
+    </inertial>
     <visual>
       <origin xyz="0 0 0" rpy="0 0 0"/>
@@ -130,4 +165,5 @@
     <limit effort="0" lower="-2.87979" upper="2.87979" velocity="4.36332"/>
     <axis xyz="0 0 1"/>
+    <dynamics damping="0.0" friction="0.0"/>
   </joint>
   <joint name="${prefix}joint_2" type="revolute">
@@ -137,4 +173,5 @@
     <limit effort="0" lower="-1.91986" upper="1.91986" velocity="4.36332"/>
     <axis xyz="0 1 0"/>
+    <dynamics damping="0.0" friction="0.0"/>
   </joint>
   <joint name="${prefix}joint_3" type="revolute">
@@ -144,4 +181,5 @@
     <limit effort="0" lower="-1.91986" upper="1.22173" velocity="4.36332"/>
     <axis xyz="0 1 0"/>
+    <dynamics damping="0.0" friction="0.0"/>
   </joint>
   <joint name="${prefix}joint_4" type="revolute">
@@ -151,4 +189,5 @@
     <limit effort="0" lower="-2.79253" upper="2.79253" velocity="7.33038"/>
     <axis xyz="1 0 0"/>
+    <dynamics damping="0.0" friction="0.0"/>
   </joint>
   <joint name="${prefix}joint_5" type="revolute">
@@ -158,4 +197,5 @@
     <limit effort="0" lower="-2.094395" upper="2.094395" velocity="10.29744"/>
     <axis xyz="0 1 0"/>
+    <dynamics damping="0.0" friction="0.0"/>
   </joint>
   <joint name="${prefix}joint_6" type="revolute">
@@ -165,4 +205,5 @@
     <limit effort="0" lower="-6.98132" upper="6.98132" velocity="10.471975"/>
     <axis xyz="1 0 0"/>
+    <dynamics damping="0.0" friction="0.0"/>
   </joint>
   <joint name="${prefix}joint6-tool0" type="fixed">

Commit message: Use plain IRB 120(T) macro as base for Gazebo model.
Avoid recursion: add '_g' suffix to Gazebo model's xacro macro name.

File: abb_irb120_gazebo/urdf/irb120.xacro (robot description, xacro)
@@ -2,4 +2,4 @@
 <robot name="abb_irb120" xmlns:xacro="http://ros.org/wiki/xacro">
   <xacro:include filename="$(find abb_irb120_gazebo)/urdf/irb120_macro.xacro"/>
-  <xacro:abb_irb120 prefix=""/>
+  <xacro:abb_irb120_g prefix=""/>
 </robot>

File: abb_irb120_gazebo/urdf/irb120_macro.xacro (robot description, xacro)
@@ -1,5 +1,8 @@
 <?xml version="1.0"?>
 <robot xmlns:xacro="http://ros.org/wiki/xacro">
-<xacro:macro name="abb_irb120" params="prefix">
+<xacro:include filename="$(find abb_irb120_support)/urdf/irb120_macro.xacro"/>
+<xacro:macro name="abb_irb120_g" params="prefix">
+  <!-- get base ABB IRB120 model -->
+  <xacro:abb_irb120 prefix="${prefix}" />
   <!-- transmission list -->
   <transmission name="${prefix}tran1">

File: abb_irb120_gazebo/urdf/irb120t.xacro (robot description, xacro)
@@ -2,4 +2,4 @@
 <robot name="abb_irb120t" xmlns:xacro="http://ros.org/wiki/xacro">
   <xacro:include filename="$(find abb_irb120_gazebo)/urdf/irb120t_macro.xacro"/>
-  <xacro:abb_irb120t prefix=""/>
+  <xacro:abb_irb120t_g prefix=""/>
 </robot>

File: abb_irb120_gazebo/urdf/irb120t_macro.xacro (robot description, xacro)
@@ -1,5 +1,8 @@
 <?xml version="1.0"?>
 <robot xmlns:xacro="http://ros.org/wiki/xacro">
-<xacro:macro name="abb_irb120t" params="prefix">
+<xacro:include filename="$(find abb_irb120_support)/urdf/irb120t_macro.xacro"/>
+<xacro:macro name="abb_irb120t_g" params="prefix">
+  <!-- get base ABB IRB120T model -->
+  <xacro:abb_irb120t prefix="${prefix}" />
   <!-- transmission list -->
   <transmission name="${prefix}tran1">

Commit message: Move Gazebo_world<->model fixed joint to top-level xacro.

File: abb_irb120_gazebo/urdf/irb120.xacro (robot description, xacro)
@@ -3,3 +3,9 @@
   <xacro:include filename="$(find abb_irb120_gazebo)/urdf/irb120_macro.xacro"/>
   <xacro:abb_irb120_g prefix=""/>
+  <!-- Fix robot to Gazebo world -->
+  <link name="world"/>
+  <joint name="world-base_link-fixed" type="fixed">
+    <parent link="world"/>
+    <child link="base_link"/>
+  </joint>
 </robot>

File: abb_irb120_gazebo/urdf/irb120_macro.xacro (robot description, xacro)
@@ -91,10 +91,4 @@
     </plugin>
   </gazebo>
-  <!-- Used for fixing robot to Gazebo world -->
-  <link name="world"/>
-  <joint name="${prefix}fixed" type="fixed">
-    <parent link="world"/>
-    <child link="${prefix}base_link"/>
-  </joint>
   </xacro:macro>
 </robot>

File: abb_irb120_gazebo/urdf/irb120t.xacro (robot description, xacro)
@@ -3,3 +3,9 @@
   <xacro:include filename="$(find abb_irb120_gazebo)/urdf/irb120t_macro.xacro"/>
   <xacro:abb_irb120t_g prefix=""/>
+  <!-- Fix robot to Gazebo world -->
+  <link name="world"/>
+  <joint name="world-base_link-fixed" type="fixed">
+    <parent link="world"/>
+    <child link="base_link"/>
+  </joint>
 </robot>

File: abb_irb120_gazebo/urdf/irb120t_macro.xacro (robot description, xacro)
@@ -91,10 +91,4 @@
     </plugin>
   </gazebo>
-  <!-- Used for fixing robot to Gazebo world -->
-  <link name="world"/>
-  <joint name="${prefix}fixed" type="fixed">
-    <parent link="world"/>
-    <child link="${prefix}base_link"/>
-  </joint>
   </xacro:macro>
 </robot>
