Commit message: modified transmission markup for indigo

File: abb_irb120_gazebo/urdf/irb120_macro.xacro (robot description, xacro)
@@ -8,7 +8,8 @@
   <transmission name="${prefix}tran1">
     <type>transmission_interface/SimpleTransmission</type>
-    <joint name="${prefix}joint_1"/>
+    <joint name="${prefix}joint_1">
+      <hardwareInterface>PositionJointInterface</hardwareInterface>
+    </joint>
     <actuator name="${prefix}motor1">
-      <hardwareInterface>PositionJointInterface</hardwareInterface>
       <mechanicalReduction>1</mechanicalReduction>
     </actuator>
@@ -16,7 +17,8 @@
   <transmission name="${prefix}tran2">
     <type>transmission_interface/SimpleTransmission</type>
-    <joint name="${prefix}joint_2"/>
+    <joint name="${prefix}joint_2">
+      <hardwareInterface>PositionJointInterface</hardwareInterface>
+    </joint>
     <actuator name="${prefix}motor2">
-      <hardwareInterface>PositionJointInterface</hardwareInterface>
       <mechanicalReduction>1</mechanicalReduction>
     </actuator>
@@ -24,7 +26,8 @@
   <transmission name="${prefix}tran3">
     <type>transmission_interface/SimpleTransmission</type>
-    <joint name="${prefix}joint_3"/>
+    <joint name="${prefix}joint_3">
+      <hardwareInterface>PositionJointInterface</hardwareInterface>
+    </joint>
     <actuator name="${prefix}motor3">
-      <hardwareInterface>PositionJointInterface</hardwareInterface>
       <mechanicalReduction>1</mechanicalReduction>
     </actuator>
@@ -32,7 +35,8 @@
   <transmission name="${prefix}tran4">
     <type>transmission_interface/SimpleTransmission</type>
-    <joint name="${prefix}joint_4"/>
+    <joint name="${prefix}joint_4">
+      <hardwareInterface>PositionJointInterface</hardwareInterface>
+    </joint>
     <actuator name="${prefix}motor4">
-      <hardwareInterface>PositionJointInterface</hardwareInterface>
       <mechanicalReduction>1</mechanicalReduction>
     </actuator>
@@ -40,7 +44,8 @@
   <transmission name="${prefix}tran5">
     <type>transmission_interface/SimpleTransmission</type>
-    <joint name="${prefix}joint_5"/>
+    <joint name="${prefix}joint_5">
+      <hardwareInterface>PositionJointInterface</hardwareInterface>
+    </joint>
     <actuator name="${prefix}motor5">
-      <hardwareInterface>PositionJointInterface</hardwareInterface>
       <mechanicalReduction>1</mechanicalReduction>
     </actuator>
@@ -48,7 +53,8 @@
   <transmission name="${prefix}tran6">
     <type>transmission_interface/SimpleTransmission</type>
-    <joint name="${prefix}joint_6"/>
+    <joint name="${prefix}joint_6">
+      <hardwareInterface>PositionJointInterface</hardwareInterface>
+    </joint>
     <actuator name="${prefix}motor6">
-      <hardwareInterface>PositionJointInterface</hardwareInterface>
       <mechanicalReduction>1</mechanicalReduction>
     </actuator>

File: abb_irb120_gazebo/urdf/irb120t_macro.xacro (robot description, xacro)
@@ -8,7 +8,8 @@
   <transmission name="${prefix}tran1">
     <type>transmission_interface/SimpleTransmission</type>
-    <joint name="${prefix}joint_1"/>
+    <joint name="${prefix}joint_1">
+      <hardwareInterface>PositionJointInterface</hardwareInterface>
+    </joint>
     <actuator name="${prefix}motor1">
-      <hardwareInterface>PositionJointInterface</hardwareInterface>
       <mechanicalReduction>1</mechanicalReduction>
     </actuator>
@@ -16,7 +17,8 @@
   <transmission name="${prefix}tran2">
     <type>transmission_interface/SimpleTransmission</type>
-    <joint name="${prefix}joint_2"/>
+    <joint name="${prefix}joint_2">
+      <hardwareInterface>PositionJointInterface</hardwareInterface>
+    </joint>
     <actuator name="${prefix}motor2">
-      <hardwareInterface>PositionJointInterface</hardwareInterface>
       <mechanicalReduction>1</mechanicalReduction>
     </actuator>
@@ -24,7 +26,8 @@
   <transmission name="${prefix}tran3">
     <type>transmission_interface/SimpleTransmission</type>
-    <joint name="${prefix}joint_3"/>
+    <joint name="${prefix}joint_3">
+      <hardwareInterface>PositionJointInterface</hardwareInterface>
+    </joint>
     <actuator name="${prefix}motor3">
-      <hardwareInterface>PositionJointInterface</hardwareInterface>
       <mechanicalReduction>1</mechanicalReduction>
     </actuator>
@@ -32,7 +35,8 @@
   <transmission name="${prefix}tran4">
     <type>transmission_interface/SimpleTransmission</type>
-    <joint name="${prefix}joint_4"/>
+    <joint name="${prefix}joint_4">
+      <hardwareInterface>PositionJointInterface</hardwareInterface>
+    </joint>
     <actuator name="${prefix}motor4">
-      <hardwareInterface>PositionJointInterface</hardwareInterface>
       <mechanicalReduction>1</mechanicalReduction>
     </actuator>
@@ -40,7 +44,8 @@
   <transmission name="${prefix}tran5">
     <type>transmission_interface/SimpleTransmission</type>
-    <joint name="${prefix}joint_5"/>
+    <joint name="${prefix}joint_5">
+      <hardwareInterface>PositionJointInterface</hardwareInterface>
+    </joint>
     <actuator name="${prefix}motor5">
-      <hardwareInterface>PositionJointInterface</hardwareInterface>
       <mechanicalReduction>1</mechanicalReduction>
     </actuator>
@@ -48,7 +53,8 @@
   <transmission name="${prefix}tran6">
     <type>transmission_interface/SimpleTransmission</type>
-    <joint name="${prefix}joint_6"/>
+    <joint name="${prefix}joint_6">
+      <hardwareInterface>PositionJointInterface</hardwareInterface>
+    </joint>
     <actuator name="${prefix}motor6">
-      <hardwareInterface>PositionJointInterface</hardwareInterface>
       <mechanicalReduction>1</mechanicalReduction>
     </actuator>
